File: Power.sch (KiCad schematic (older format))
At the start: 64 parts, among them J3 Conn_01x02, J4 Conn_01x02, J5 Conn_ARM_JTAG_SWD_10, Q1 MMBT5401LT1G, Q2 Q_NMOS_GDS, Q3 MMBT3904, Q4 Q_NMOS_GDS, Q5 Q_NMOS_GDS, Q6 Q_NMOS_GDS, U10 LMZ21700SIL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

Commit message: Changed connectors to microfit, added fan output
Parts:
- added J7: FAN, Connector_Molex:Molex_KK-254_AE-6410-03A_1x03_P2.54mm_Vertical, symbol Connector_Generic:Conn_01x03
- J3: value Conn_01x02 -> ESTOP; footprint Connector_Molex:Molex_Nano-Fit_105313-xx02_1x02_P2.50mm_Horizontal -> BLDC:molex-0436500213; symbol Connector_Generic:Conn_01x02 -> Connector_Generic:Conn_01x04
- J4: value Conn_01x02 -> PWR; footprint Connectors_OSRF:PP45_1X2 -> BLDC:molex-0436500213; symbol Connector_Generic:Conn_01x02 -> Connector_Generic:Conn_01x04
- R14: value 2m -> 15m
Connections:
- net +12V: now also J7.2 (Pin_2)
- net GNDPWR: now also J3.2 (Pin_2), J3.3 (Pin_3), J3.4 (Pin_4), J4.3 (Pin_3), J4.4 (Pin_4), J7.1 (Pin_1); no longer J3.1 (Pin_1), U6.24 (nRETRY)
- net LM_VDD: now reaches C30.1, U6.21 (VDD)
- net LM_VDD: now also U6.24 (nRETRY)
- net at R12.2, R13.1, U6.7 (UVLO): now also J3.1 (Pin_1); no longer J3.2 (Pin_2)
- no-connect marks 9 -> 10
Other:
- moved on the sheet: C27, C28, C29, C30, C31, C32, C36, C38, C39, C40, C41, C42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
