File: hardware/blue_interface_board.kicad_pcb (KiCad board)
At the start: 4 copper layers, 70 x 70 mm, 130 parts, among them J1 arm connector, J10 I2C, J2 USB_B_Micro, J3 ESTOP, J4 PWR, J5 Conn_ARM_JTAG_SWD_10, J6 logic-side RS485 debug/expans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, J7 FAN, J8 power-side RS485 debug/expans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, J9 DEBUG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

Commit message: Updating date
Other:
- board text added: "DEC 2020"
- board text removed: "FEB 2020"
Changed lines of the file:
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@@
     (effects (font (size 1.8 1.8) (thickness 0.3)))
   )
-  (gr_text "FEB 2020" (at 108 64.3) (layer "F.SilkS")
+  (gr_text "DEC 2020" (at 108 64.3) (layer "F.SilkS")
     (effects (font (size 1.8 1.8) (thickness 0.3)))
   )
